File: readout/board/hp8565-readout/hp8565-readout.kicad_pcb (KiCad board)
At the start: 4 copper layers, 78.7 x 30.5 mm, 20 parts, among them J1 Pin_Header, J2 Pin_Header, J3 DIP Socket, J4 Pin_Header, J5 Masach_MS230-20S, P1 DIP Pins, U1 ATmega4809-M, U2 GD75232DB

Commit message: Route CF connector.
Parts:
- moved C2 1.27 mm to (152.7, 91.4)
Connections:
- J3 pad 12: /HCF1 -> /CF1
- J3 pad 13: /HCF2 -> /CF2
- J3 pad 15: /HCF4 -> /CF4
- J3 pad 16: /HCF5 -> /CF5
- J3 pad 6: /LCF3 -> /~{CF3}
- J3 pad 7: /LCF0 -> /~{CF0}
- P1 pad 12: /HCF1 -> /CF1
- P1 pad 13: /HCF2 -> /CF2
- P1 pad 15: /HCF4 -> /CF4
- P1 pad 16: /HCF5 -> /CF5
- P1 pad 6: /LCF3 -> /~{CF3}
- P1 pad 7: /LCF0 -> /~{CF0}
- U1 pad 11: unconnected-(U1-Pad11) -> /dpC
- U1 pad 12: unconnected-(U1-Pad12) -> /~{CF0}
- U1 pad 13: unconnected-(U1-Pad13) -> /CF1
- U1 pad 16: unconnected-(U1-Pad16) -> /CF2
- U1 pad 17: unconnected-(U1-Pad17) -> /~{CF3}
- U1 pad 18: unconnected-(U1-Pad18) -> /CF4
- U1 pad 19: unconnected-(U1-Pad19) -> /CF5
- U1 pad 20: unconnected-(U1-Pad20) -> /CFa
- U1 pad 21: unconnected-(U1-Pad21) -> /CFb
- U1 pad 22: unconnected-(U1-Pad22) -> /CFc
- U1 pad 23: unconnected-(U1-Pad23) -> /CFd
- U1 pad 24: unconnected-(U1-Pad24) -> /CFe
- U1 pad 25: unconnected-(U1-Pad25) -> /CFf
- U1 pad 26: unconnected-(U1-Pad26) -> /CFg
- U1 pad 27: unconnected-(U1-Pad27) -> /CFdp
Routing:
- net /CF5: track 0.00 -> 46.3 mm, vias 0 -> 1
- net /CF4: track 0.00 -> 44.2 mm, vias 0 -> 1
- net /CF2: track 0.00 -> 39.7 mm, vias 0 -> 1
- net /CF1: track 0.00 -> 38.5 mm, vias 0 -> 1
- net /~{CF0}: track 0.00 -> 35.9 mm, vias 0 -> 1
- net /~{CF3}: track 0.00 -> 35.0 mm, vias 0 -> 1
- net /CFdp: track 15.0 -> 44.2 mm, vias 0 -> 1
- net /CFf: track 15.0 -> 43.2 mm, vias 0 -> 1
- net /CFg: track 15.0 -> 39.7 mm, vias 0 -> 1
- net /CFa: track 15.0 -> 38.7 mm, vias 0 -> 1
- net /dpC: track 15.0 -> 37.5 mm, vias 0 -> 1
- net /CFe: track 15.0 -> 35.4 mm, vias 0 -> 1
- net /CFd: track 15.0 -> 33.2 mm, vias 0 -> 1
- net /CFb: track 15.0 -> 33.1 mm, vias 0 -> 1
- net /LCF0: track 15.0 -> 0.00 mm
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
Commit message: Clean up silkscreen and stuff.
Parts:
- added R1: 1k5, Resistor_SMD:R_0402_1005Metric, F.Cu at (113.5, 77.5)
- renumbered R1 to R5
Routing:
- net GND: track 37.4 -> 48.2 mm, vias 48 -> 61
- net /LOG/~{LIN}: track 42.9 -> 45.2 mm
- net /CK: track 51.4 -> 53.2 mm
- net /CFc: track 26.7 -> 25.4 mm
- net +15V: track 42.3 -> 41.2 mm
- net /LTXD: track 21.4 -> 22.1 mm
- net /CFf: track 43.2 -> 42.6 mm
- net /UPDI: track 50.2 -> 50.8 mm
- added copper zone on B.Cu, net GND
Other:
- board text added: "R1..4"
